File: tamagotchi.kicad_pcb (KiCad board)
At the start: 2 copper layers, 55 x 80 mm, 9 parts, among them SW1 SW_Push, SW2 SW_Push, SW3 SW_Push, U1 XIAO-ESP32-C3-SMD, U2 HS96L03W2C03

Commit message: Add files via upload
Other:
- board size 55 x 80 mm -> 48 x 87 mm
Changed lines of the file:
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@@
 		(pad "" np_thru_hole circle
 			(at 0 0)
-			(size 3.2 3.2)
-			(drill 3.2)
+			(size 2.1 2.1)
+			(drill 2.1)
 			(layers "*.Cu" "*.Mask")
 		)
@@
 		(pad "" np_thru_hole circle
 			(at 0 0)
-			(size 3.2 3.2)
-			(drill 3.2)
+			(size 2.1 2.1)
+			(drill 2.1)
 			(layers "*.Cu" "*.Mask")
 		)
@@
 		(embedded_fonts no)
 	)
-	(gr_poly
-		(pts
-			(xy 143.5 54) (xy 118 54) (xy 108.5 64) (xy 103.5 74) (xy 103 114) (xy 108 123.5) (xy 118 134) (xy 143 134)
-			(xy 153 124) (xy 158 114) (xy 158 73.5) (xy 153.5 64)
-		)
+	(gr_line
+		(start 106.5 72)
+		(end 126.5 52)
 		(stroke
-			(width 0.5)
-			(type solid)
-		)
-		(fill no)
+			(width 0.2)
+			(type default)
+		)
 		(layer "Edge.Cuts")
 	)
+	(gr_line
+		(start 106.5 119)
+		(end 106.5 72)
+		(stroke
+			(width 0.2)
+			(type default)
+		)
+		(layer "Edge.Cuts")
+	)
+	(gr_line
+		(start 106.5 119)
+		(end 126.5 139)
+		(stroke
+			(width 0.2)
+			(type default)
+		)
+		(layer "Edge.Cuts")
+	)
+	(gr_line
+		(start 126.5 52)
+		(end 134.5 52)
+		(stroke
+			(width 0.2)
+			(type default)
+		)
+		(layer "Edge.Cuts")
+	)
+	(gr_line
+		(start 126.5 139)
+		(end 134.5 139)
+		(stroke
+			(width 0.2)
+			(type default)
+		)
+		(layer "Edge.Cuts")
+	)
+	(gr_line
+		(start 134.5 139)
+		(end 154.5 119)
+		(stroke
+			(width 0.2)
+			(type default)
+		)
+		(layer "Edge.Cuts")
+	)
+	(gr_line
+		(start 154.5 72)
+		(end 134.5 52)
+		(stroke
+			(width 0.2)
+			(type default)
+		)
+		(layer "Edge.Cuts")
+	)
+	(gr_line
+		(start 154.5 119)
+		(end 154.5 72)
+		(stroke
+			(width 0.2)
+			(type default)
+		)
+		(layer "Edge.Cuts")
+	)
